File: GoPack Board Rev A/Pi MCU shield.brd (EAGLE design)
At the start: 73 x 65 mm, 63 parts, among them U1 DSPIC33FJ64MC204TQFP, U2 LMH6644MT, U3 LMH6644MT, U4 MC3846D, U5 UA9637AC, U6 LM25011, U7 5V Reg, U8 3V3 Reg, U9 LMH6644MT, X1 Supply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

Commit message: Updated board files 2-24-17
Parts:
- JP3: device pinhead:2X07 -> pinhead:2X10
- R9: value 9.1k -> 4.7k
- moved JP3 2.50 mm to (30.5, 51.9)
Connections:
- removed net +10V: C11.1, C14.1, JP3.10, JP3.9, L1.P$2, R13.2, R9.2, U7.3
- removed net N$40: R11.1, U6.7
- new net +6V3: C11.1, C14.1, JP3.17, JP3.19, L1.P$2, R13.2, R9.2, U7.3
- net +3V3: now also JP3.5, JP3.7; no longer JP3.2, JP3.4
- net +5V: now also JP3.11, JP3.13, JP3.15, JP3.9; no longer JP3.5, JP3.6, JP3.7, JP3.8
- net GND: now also JP3.10, JP3.16, JP3.18, JP3.2, JP3.20, JP3.4, JP3.6, JP3.8, R11.1, U6.7; no longer JP3.11, JP3.13, R14.1, R15.1, R16.1, R5.1, R6.1, R7.1
Routing:
- net +10V: track 92.4 -> 0.00 mm, vias 8 -> 0
- net +6V3: track 0.00 -> 85.8 mm, vias 0 -> 8
- net N$40: track 6.30 -> 0.00 mm
- net GND: track 122.9 -> 117.2 mm, vias 27 -> 26
- net +5V: track 124.9 -> 119.6 mm
- net +3V3: track 156.3 -> 152.9 mm
- net N$3: track 24.5 -> 22.3 mm
- net N$35: track 5.13 -> 4.23 mm
- added copper zone on layer 1, net +6V3
- removed copper zone on layer 1, net +10V
Other:
- board text added: "+6V3"
- board text added: "+Vdd"
- board text removed: "+10V"
