File: GoPack Board Rev A/Pi MCU shield.sch (EAGLE design)
At the start: 63 parts, among them U1 DSPIC33FJ64MC204TQFP, U2 LMH6644MT, U3 LMH6644MT, U4 MC3846D, U5 UA9637AC, U6 LM25011, U7 5V Reg, U8 3V3 Reg, U9 LMH6644MT, X1 Supply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

Commit message: Updated board files 2-24-17
Parts:
- JP3: device pinhead:PINHD-2X7 -> pinhead:PINHD-2X10
- R9: value 9.1k -> 4.7k
Connections:
- removed net +10V: C11.1, C14.1, JP3.10, JP3.9, L1.2, R13.2, R9.2, U7.IN
- removed net N$40: R11.1, U6.CSG
- new net +6V3: C11.1, C14.1, JP3.17, JP3.19, L1.2, R13.2, R9.2, U7.IN
- net +3V3: now also JP3.5, JP3.7; no longer JP3.2, JP3.4
- net +5V: now also JP3.11, JP3.13, JP3.15, JP3.9; no longer JP3.5, JP3.6, JP3.7, JP3.8
- net GND: now also JP3.10, JP3.16, JP3.18, JP3.2, JP3.20, JP3.4, JP3.6, JP3.8, R11.1, U6.CSG; no longer JP3.11, JP3.13, R14.A, R15.A, R16.A, R5.A, R6.A, R7.A

Commit message: Updated board files
Parts:
- removed R17, R18, R19: 1k, resistor:R-US_R0603
- R14, R15, R16: value 10k -> 50k
- R2, R8: value 150 -> 1k
- R3, R4: value 82 -> 470
Connections:
- net GND: now also R14.A, R15.A, R16.A; no longer R17.1, R18.1, R19.1
- net N$1: no longer R18.2
- net N$10: no longer R17.2
- net N$31: no longer R19.2
Changed lines of the file:
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@@
 <part name="P+9" library="supply1" deviceset="+5V" device=""/>
 <part name="LED1" library="led" deviceset="LTST-C19HE1WT" device=""/>
-<part name="R2" library="resistor" deviceset="R-US_" device="R0603" value="150"/>
-<part name="R3" library="resistor" deviceset="R-US_" device="R0603" value="82"/>
-<part name="R4" library="resistor" deviceset="R-US_" device="R0603" value="82"/>
-<part name="R8" library="resistor" deviceset="R-US_" device="R0603" value="150"/>
+<part name="R2" library="resistor" deviceset="R-US_" device="R0603" value="1k"/>
+<part name="R3" library="resistor" deviceset="R-US_" device="R0603" value="470"/>
+<part name="R4" library="resistor" deviceset="R-US_" device="R0603" value="470"/>
+<part name="R8" library="resistor" deviceset="R-US_" device="R0603" value="1k"/>
 <part name="LED2" library="led" deviceset="LED" device="SML0603" value="Yellow"/>
 <part name="U9" library="texas" deviceset="LMH6644" device="MT"/>
-<part name="R14" library="rcl" deviceset="R-TRIMM" device="3224J" value="10k"/>
-<part name="R15" library="rcl" deviceset="R-TRIMM" device="3224J" value="10k"/>
-<part name="R16" library="rcl" deviceset="R-TRIMM" device="3224J" value="10k"/>
-<part name="R17" library="resistor" deviceset="R-US_" device="R0603" value="1k"/>
-<part name="R18" library="resistor" deviceset="R-US_" device="R0603" value="1k"/>
-<part name="R19" library="resistor" deviceset="R-US_" device="R0603" value="1k"/>
+<part name="R14" library="rcl" deviceset="R-TRIMM" device="3224J" value="50k"/>
+<part name="R15" library="rcl" deviceset="R-TRIMM" device="3224J" value="50k"/>
+<part name="R16" library="rcl" deviceset="R-TRIMM" device="3224J" value="50k"/>
 <part name="+3V8" library="supply1" deviceset="+3V3" device=""/>
 <part name="GND14" library="supply1" deviceset="GND" device=""/>
@@
 <instance part="R15" gate="G$1" x="109.22" y="2.54"/>
 <instance part="R16" gate="G$1" x="109.22" y="-17.78"/>
-<instance part="R17" gate="G$1" x="119.38" y="17.78" rot="R90"/>
-<instance part="R18" gate="G$1" x="119.38" y="-2.54" rot="R90"/>
-<instance part="R19" gate="G$1" x="119.38" y="-22.86" rot="R90"/>
 <instance part="+3V8" gate="G$1" x="157.48" y="30.48"/>
 <instance part="GND14" gate="1" x="167.64" y="-8.636"/>
@@
 </segment>
 <segment>
-<pinref part="R19" gate="G$1" pin="1"/>
-<wire x1="119.38" y1="-27.94" x2="119.38" y2="-30.48" width="0.1524" layer="91"/>
 <pinref part="GND15" gate="1" pin="GND"/>
+<pinref part="R16" gate="G$1" pin="A"/>
+<wire x1="109.22" y1="-22.86" x2="119.38" y2="-22.86" width="0.1524" layer="91"/>
+<wire x1="119.38" y1="-22.86" x2="119.38" y2="-30.48" width="0.1524" layer="91"/>
 </segment>
 <segment>
 <pinref part="GND25" gate="1" pin="GND"/>
-<pinref part="R18" gate="G$1" pin="1"/>
-<wire x1="119.38" y1="-7.62" x2="114.3" y2="-7.62" width="0.1524" layer="91"/>
+<pinref part="R15" gate="G$1" pin="A"/>
+<wire x1="109.22" y1="-2.54" x2="114.3" y2="-2.54" width="0.1524" layer="91"/>
+<wire x1="114.3" y1="-2.54" x2="114.3" y2="-7.62" width="0.1524" layer="91"/>
 </segment>
 <segment>
 <pinref part="GND26" gate="1" pin="GND"/>
-<pinref part="R17" gate="G$1" pin="1"/>
-<wire x1="119.38" y1="12.7" x2="114.3" y2="12.7" width="0.1524" layer="91"/>
-<wire x1="114.3" y1="12.7" x2="114.3" y2="10.16" width="0.1524" layer="91"/>
+<pinref part="R14" gate="G$1" pin="A"/>
+<wire x1="109.22" y1="17.78" x2="114.3" y2="17.78" width="0.1524" layer="91"/>
+<wire x1="114.3" y1="17.78" x2="114.3" y2="10.16" width="0.1524" layer="91"/>
 </segment>
 <segment>
@@
 <segment>
 <pinref part="R14" gate="G$1" pin="S"/>
-<pinref part="R17" gate="G$1" pin="2"/>
-<wire x1="114.3" y1="22.86" x2="119.38" y2="22.86" width="0.1524" layer="91"/>
-<wire x1="119.38" y1="22.86" x2="129.54" y2="22.86" width="0.1524" layer="91"/>
+<wire x1="114.3" y1="22.86" x2="129.54" y2="22.86" width="0.1524" layer="91"/>
 <wire x1="129.54" y1="22.86" x2="129.54" y2="7.62" width="0.1524" layer="91"/>
-<junction x="119.38" y="22.86"/>
 <pinref part="U9" gate="U1" pin="+INA"/>
 <wire x1="129.54" y1="7.62" x2="152.4" y2="7.62" width="0.1524" layer="91"/>
@@
 <net name="N$31" class="0">
 <segment>
-<pinref part="R19" gate="G$1" pin="2"/>
 <pinref part="R16" gate="G$1" pin="S"/>
-<wire x1="119.38" y1="-17.78" x2="114.3" y2="-17.78" width="0.1524" layer="91"/>
-<wire x1="119.38" y1="-17.78" x2="142.24" y2="-17.78" width="0.1524" layer="91"/>
+<wire x1="114.3" y1="-17.78" x2="142.24" y2="-17.78" width="0.1524" layer="91"/>
 <wire x1="142.24" y1="-17.78" x2="142.24" y2="-12.7" width="0.1524" layer="91"/>
-<junction x="119.38" y="-17.78"/>
 <pinref part="U9" gate="U1" pin="+INC"/>
 <wire x1="142.24" y1="-12.7" x2="152.4" y2="-12.7" width="0.1524" layer="91"/>
@@
 <segment>
 <pinref part="R15" gate="G$1" pin="S"/>
-<pinref part="R18" gate="G$1" pin="2"/>
 <wire x1="114.3" y1="2.54" x2="119.38" y2="2.54" width="0.1524" layer="91"/>
 <wire x1="119.38" y1="2.54" x2="119.38" y2="5.08" width="0.1524" layer="91"/>
-<junction x="119.38" y="2.54"/>
 <pinref part="U9" gate="U1" pin="+INB"/>
 <wire x1="162.56" y1="7.62" x2="180.34" y2="7.62" width="0.1524" layer="91"/>
